File: pcb/matrix.kicad_sch (KiCad schematic)
At the start: 143 parts

Commit message: Trace updates
Parts:
- added MX77: 1.5u, Alps_Only:ALPS-1.5U, symbol Switch:SW_SPST
Connections:
- net COL0: now also MX77.2 (B)
- net at D32.2 (A), MX33.1 (A), MX34.1 (A): now also MX77.1 (A)
Changed lines of the file:
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@@
   (junction (at 185.42 39.37) (diameter 0) (color 0 0 0 0)
   )
+  (junction (at 31.75 80.645) (diameter 0) (color 0 0 0 0)
+  )
   (junction (at 209.55 118.11) (diameter 0) (color 0 0 0 0)
   )
@@
   (junction (at 143.51 74.93) (diameter 0) (color 0 0 0 0)
   )
+  (junction (at 41.91 74.93) (diameter 0) (color 0 0 0 0)
+  )
   (junction (at 73.66 74.93) (diameter 0) (color 0 0 0 0)
   )
@@
     (stroke (width 0) (type default) (color 0 0 0 0))
   )
+  (wire (pts (xy 41.91 74.93) (xy 41.91 80.645))
+    (stroke (width 0) (type default) (color 0 0 0 0))
+  )
   (wire (pts (xy 83.82 46.99) (xy 69.85 46.99))
     (stroke (width 0) (type default) (color 0 0 0 0))
@@
     (stroke (width 0) (type default) (color 0 0 0 0))
   )
-  (wire (pts (xy 31.75 74.93) (xy 31.75 85.09))
+  (wire (pts (xy 31.75 74.93) (xy 31.75 80.645))
     (stroke (width 0) (type default) (color 0 0 0 0))
   )
@@
     (stroke (width 0) (type default) (color 0 0 0 0))
   )
+  (wire (pts (xy 31.75 80.645) (xy 31.75 85.09))
+    (stroke (width 0) (type default) (color 0 0 0 0))
+  )
   (wire (pts (xy 97.79 82.55) (xy 83.82 82.55))
     (stroke (width 0) (type default) (color 0 0 0 0))
@@
       (effects (font (size 1.27 1.27)) hide)
     )
+    (pin "1")
+    (pin "2")
+  )
+  (symbol (lib_id "Switch:SW_SPST") (at 36.83 80.645 0) (mirror y) (unit 1)
+    (in_bom yes) (on_board yes)
+    (property "Reference" "MX77" (id 0) (at 36.83 74.676 0))
+    (property "Value" "1.5u" (id 1) (at 36.83 76.9874 0))
+    (property "Footprint" "Alps_Only:ALPS-1.5U" (id 2) (at 36.83 80.645 0)
+      (effects (font (size 1.27 1.27)) hide)
+    )
+    (property "Datasheet" "~" (id 3) (at 36.83 80.645 0)
+      (effects (font (size 1.27 1.27)) hide)
+    )
